File: mpw-mb1.kicad_pcb (KiCad board)
At the start: 2 copper layers, 62 x 90 mm, 128 parts, among them CON1 95157-440LF, CON2 95157-440LF, J1 USB_C_Receptacle_USB2.0, J2 Conn_01x02, J3 Conn_01x03, J4 Conn_01x06, J5 Conn_01x22, J6 Conn_01x22, J7 Conn_01x02, SW1 SW_Push, U1 MCP1319, U2 MIC5318, U3 AZ1117-3.3, U4 W25Q32JVSS, U5 Pico, X1 10MHz

Commit message: basic placement started
Parts:
- removed C1, C10, C11, C12, C13, C14, C15, C16, C17: 100nF, Capacitor_SMD:C_0603_1608Metric
- removed CON1, CON2: 95157-440LF, Connector_PinHeader_2.54mm:PinHeader_2x20_P2.54mm_Vertical_SMD
- removed RV1: 1k, Potentiometer_SMD:Potentiometer_Bourns_TC33X_Vertical
- removed the U1 at (13.0, -18.8)
- removed U2: MIC5318, Package_TO_SOT_SMD:SOT-23-5
- removed kibuzzard-64038B6B: G***, kibuzzard-64038B6B
- added C18: 100nF, Capacitor_SMD:C_0603_1608Metric, F.Cu at (115.8, 117.5)
- added C19: 100nF, Capacitor_SMD:C_0603_1608Metric, F.Cu at (115.8, 79.5)
- added C20: 100nF, Capacitor_SMD:C_0603_1608Metric, F.Cu at (115.8, 112.3)
- added C21: 100nF, Capacitor_SMD:C_0603_1608Metric, F.Cu at (115.8, 82.2)
- added C22: 100nF, Capacitor_SMD:C_0603_1608Metric, F.Cu at (115.8, 114.9)
- added C23: 100nF, Capacitor_SMD:C_0603_1608Metric, F.Cu at (115.8, 110.0)
- added C24: 100nF, Capacitor_SMD:C_0603_1608Metric, F.Cu at (115.8, 76.9)
- added C25: 10uF, Capacitor_SMD:C_0603_1608Metric, F.Cu at (221.2, 227.0)
- added C26: 10uF, Capacitor_SMD:C_0603_1608Metric, F.Cu at (225.2, 209.5)
- added C27: 100nF, Capacitor_SMD:C_0603_1608Metric, F.Cu at (117.0, 127.7)
- added C28: 1uF, Capacitor_SMD:C_0603_1608Metric, F.Cu at (117.0, 126.2)
- added C29: 100nF, Capacitor_SMD:C_0603_1608Metric, F.Cu at (91.8, 127.4)
- added C30: 1uF, Capacitor_SMD:C_0603_1608Metric, F.Cu at (91.8, 125.9)
- added C31: 1uF, Capacitor_SMD:C_0603_1608Metric, F.Cu at (225.2, 222.0)
- added C32: 1uF, Capacitor_SMD:C_0603_1608Metric, F.Cu at (225.2, 224.5)
- added C33: 10uF, Capacitor_SMD:C_0805_2012Metric, F.Cu at (41.5, 155.4)
- added C34: 22uF, Capacitor_SMD:C_0805_2012Metric, F.Cu at (41.7, 143.1)
- added C35: 100nF, Capacitor_SMD:C_0603_1608Metric, F.Cu at (41.8, 141.2)
- added FID1: Fiducial, Fiducial:Fiducial_1mm_Mask2mm, F.Cu at (152.9, 7.90)
- added FID2: Fiducial, Fiducial:Fiducial_1mm_Mask2mm, F.Cu at (152.9, 11.4)
- added FID3: Fiducial, Fiducial:Fiducial_1mm_Mask2mm, F.Cu at (152.9, 15.0)
- added J10: 613012243121, TinyTapeout:PinSocket_2x06_P2.54mm_PMODHost1A, F.Cu at (91.1, 130.3)
- added J11: Conn_02x02_Odd_Even, Connector_PinHeader_2.54mm:PinHeader_2x02_P2.54mm_Vertical, F.Cu at (75.2, 126.3)
- added J8: Conn_01x22, Connector_PinHeader_2.54mm:PinHeader_1x22_P2.54mm_Vertical, B.Cu at (195.6, 64.3)
- added J9: 613012243121, TinyTapeout:PinSocket_2x06_P2.54mm_PMODHost1A, F.Cu at (116.1, 130.6)
- added JP1: SolderJumper_2_Bridged, TinyTapeout:SolderJumper-2_Bridged_Throughole1, F.Cu at (134.8, 115.9)
- added JP2: SolderJumper_2_Bridged, TinyTapeout:SolderJumper-2_Bridged_Throughole1, F.Cu at (134.8, 118.4)
- added JP3: SolderJumper_2_Bridged, TinyTapeout:SolderJumper-2_Bridged_Throughole1, F.Cu at (134.8, 120.9)
- added JP4: SolderJumper_2_Bridged, TinyTapeout:SolderJumper-2_Bridged_Throughole1, F.Cu at (134.8, 123.4)
- added JP5: SolderJumper_2_Bridged, TinyTapeout:SolderJumper-2_Bridged_Throughole1, F.Cu at (134.8, 125.9)
- added JP6: SolderJumper_2_Bridged, TinyTapeout:SolderJumper-2_Bridged_Throughole1, F.Cu at (134.8, 128.4)
- added JP7: SolderJumper_2_Bridged, TinyTapeout:SolderJumper-2_Bridged_Throughole1, F.Cu at (134.8, 130.9)
- added JP8: SolderJumper_2_Bridged, TinyTapeout:SolderJumper-2_Bridged_Throughole1, F.Cu at (134.8, 133.4)
- added R15: 68R, Resistor_SMD:R_0603_1608Metric, F.Cu at (138.5, 115.9)
- added R16: 68R, Resistor_SMD:R_0603_1608Metric, F.Cu at (138.5, 118.4)
- added R17: 68R, Resistor_SMD:R_0603_1608Metric, F.Cu at (138.5, 120.9)
- added R18: 68R, Resistor_SMD:R_0603_1608Metric, F.Cu at (138.5, 123.4)
- added R19: 68R, Resistor_SMD:R_0603_1608Metric, F.Cu at (138.5, 125.9)
- added R20: 68R, Resistor_SMD:R_0603_1608Metric, F.Cu at (138.5, 128.4)
- added R21: 68R, Resistor_SMD:R_0603_1608Metric, F.Cu at (138.5, 130.9)
- added R22: 68R, Resistor_SMD:R_0603_1608Metric, F.Cu at (138.5, 133.4)
- added R23: 10k, Resistor_SMD:R_0603_1608Metric, F.Cu at (83.7, 87.0)
- added R24: 10k, Resistor_SMD:R_0603_1608Metric, F.Cu at (83.7, 84.5)
- added R25: 10k, Resistor_SMD:R_0603_1608Metric, F.Cu at (83.7, 82.0)
- added R26: 10k, Resistor_SMD:R_0603_1608Metric, F.Cu at (83.7, 79.4)
- added R27: 10k, Resistor_SMD:R_0603_1608Metric, F.Cu at (83.7, 76.9)
- added R28: 10k, Resistor_SMD:R_0603_1608Metric, F.Cu at (83.7, 74.4)
- added R29: 10k, Resistor_SMD:R_0603_1608Metric, F.Cu at (83.7, 71.9)
- added R30: 10k, Resistor_SMD:R_0603_1608Metric, F.Cu at (83.7, 69.4)
- added R31: 510, Resistor_SMD:R_0603_1608Metric, F.Cu at (237.2, 209.5)
- added R32: 10k, Resistor_SMD:R_0603_1608Metric, F.Cu at (72.5, 59.1)
- added R34: 1.2K, Resistor_SMD:R_0603_1608Metric, F.Cu at (71.0, 59.1)
- added R39: 10k, Resistor_SMD:R_0603_1608Metric, F.Cu at (237.2, 217.0)
- added R49: 10k, Resistor_SMD:R_0603_1608Metric, F.Cu at (92.5, 64.4)
- added RN1: 10k, Resistor_SMD:R_Array_Convex_8x0602, F.Cu at (76.7, 120.4)
- added RN2: 10k, Resistor_SMD:R_Array_Convex_8x0602, F.Cu at (76.3, 64.4)
- added SW2: 418121270808, TinyTapeout:418121270808, F.Cu at (75.0, 78.2)
- added SW3: 219-9MST, TinyTapeout:219-9GULLWING, F.Cu at (75.2, 103.3)
- added SW5: B3U-1000P, Button_Switch_SMD:SW_SPST_B3U-1000P, F.Cu at (89.9, 64.4)
- added TP10: TestPoint, TestPoint:TestPoint_Pad_D1.5mm, F.Cu at (141.1, 82.7)
- added TP11: TestPoint, TestPoint:TestPoint_Pad_D1.5mm, F.Cu at (138.5, 78.8)
- added TP12: TestPoint, TestPoint:TestPoint_Pad_D1.5mm, F.Cu at (133.1, 94.5)
- added TP13: TestPoint, TestPoint:TestPoint_Pad_D1.5mm, F.Cu at (81.5, 63.9)
- added TP4: Keystone 5019, TestPoint:TestPoint_Keystone_5019_Minature, F.Cu at (212.8, 228.2)
- added TP5: Keystone 5019, TestPoint:TestPoint_Keystone_5019_Minature, F.Cu at (212.8, 232.2)
- added TP6: TestPoint, TestPoint:TestPoint_Pad_D1.5mm, F.Cu at (76.1, 58.3)
- added TP7: TestPoint, TestPoint:TestPoint_Pad_D1.5mm, F.Cu at (135.9, 78.9)
- added TP8: TestPoint, TestPoint:TestPoint_Pad_D1.5mm, F.Cu at (141.0, 94.6)
- added TP9: TestPoint, TestPoint:TestPoint_Pad_D1.5mm, F.Cu at (136.7, 98.3)
- added U6: AZ1117-1.8, Package_TO_SOT_SMD:SOT-223-3_TabPin2, F.Cu at (39.6, 149.4)
- added U7: 157112V12700, Display_7Segment:KCSC02-106, F.Cu at (144.5, 124.6)
- C2, C7: value 1uF -> 100nF
- C4: value DNP -> 6800pF
- J1: value USB_C_Receptacle_USB2.0 -> TT03_BREAKOUT; footprint Connector_USB:USB_C_Receptacle_HRO_TYPE-C-31-M-12 -> TinyTapeout:TT03_BREAKOUT_SMB
- J2: value Conn_01x02 -> USB_C_Receptacle_USB2.0; footprint Connector_PinHeader_2.54mm:PinHeader_1x02_P2.54mm_Vertical -> Connector_USB:USB_C_Receptacle_HRO_TYPE-C-31-M-12
- J3: value Conn_01x03 -> Conn_01x02; footprint Connector_PinHeader_2.54mm:PinHeader_1x03_P2.54mm_Vertical -> Connector_PinHeader_2.54mm:PinHeader_1x02_P2.54mm_Vertical
- J4: value Conn_01x06 -> Conn_01x03; footprint Connector_PinHeader_2.54mm:PinHeader_1x06_P2.54mm_Vertical -> Connector_PinHeader_2.54mm:PinHeader_1x03_P2.54mm_Vertical
- J5: value Conn_01x22 -> Conn_01x03; footprint Connector_PinHeader_2.54mm:PinHeader_1x22_P2.54mm_Vertical -> Connector_PinHeader_2.54mm:PinHeader_1x03_P2.54mm_Vertical; moved to F.Cu
- J6: value Conn_01x22 -> Conn_01x06; footprint Connector_PinHeader_2.54mm:PinHeader_1x22_P2.54mm_Vertical -> Connector_PinHeader_2.54mm:PinHeader_1x06_P2.54mm_Vertical; moved to F.Cu
- J7: value Conn_01x02 -> Conn_01x22; footprint Connector_PinHeader_2.54mm:PinHeader_1x02_P2.54mm_Vertical -> Connector_PinHeader_2.54mm:PinHeader_1x22_P2.54mm_Vertical; moved to B.Cu
- R5: value 1k -> 1M
- R6: value 4.3k -> 10k
- SW1: value SW_Push -> B3U-1000P
- U1: renamed from U5; footprint pico:RPi_Pico_SMD -> RPi_Pico:RPi_Pico_SMD
- moved D4 307.8 mm to (47.9, 226.8), turned to 0 degrees
- moved R14 303.9 mm to (50.9, 226.8)
- moved R11 253.4 mm to (51.0, 231.2), turned to 180 degrees
- moved R12 251.4 mm to (50.9, 228.9), turned to 180 degrees
- moved D1 249.5 mm to (48.0, 231.2), turned to 0 degrees
- moved R13 247.9 mm to (50.9, 224.9), turned to 180 degrees
- moved D2 247.5 mm to (47.9, 228.9), turned to 0 degrees
- moved D3 243.9 mm to (47.9, 224.9), turned to 0 degrees
- moved J2 242.8 mm to (36.1, 170.7), turned to 0 degrees
- moved R7 195.9 mm to (138.2, 95.3), turned to 90 degrees
- moved J4 195.9 mm to (-10.7, 102.3), turned to -90 degrees
- moved R10 193.9 mm to (136.7, 95.3), turned to 90 degrees
- moved R9 192.1 mm to (139.0, 81.8), turned to -90 degrees
- moved R3 191.9 mm to (135.2, 95.3), turned to 90 degrees
- moved U4 191.2 mm to (136.7, 88.6), turned to 90 degrees
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Connections:
- net ~{MEM_HOLD} renamed Net-(U4-IO3)
- net ~{MEM_WP} renamed Net-(U4-IO2)
- C2 pad 1: vdda -> ext_clk
- C4 pad 1: Net-(C4-Pad1) -> Net-(J2-SHIELD)
- C5 pad 2: vdda -> +3.3V
- C6 pad 1: vdda -> +3.3V
- C7 pad 1: vccd -> +3.3V
- C7 pad 2: GND -> RST
- C8 pad 1: vdda -> +3.3V
- C9 pad 2: vdda -> +3.3V
- J1 pad A12: GND -> mprj_io6_ser_tx
- J1 pad A4: VBUS -> +1V8
- J1 pad A5: Net-(J1-PadA5) -> GND
- J1 pad A6: unconnected-(J1-PadA6) -> +3.3V
- J1 pad A7: unconnected-(J1-PadA7) -> GND
- J1 pad A8: unconnected-(J1-PadA8) -> +1V8
- J1 pad A9: VBUS -> GND
- J1 pad B4: VBUS -> scansel0
- J1 pad B5: Net-(J1-PadB5) -> set_clk_div
- J1 pad B6: unconnected-(J1-PadB6) -> slow_clk
- J1 pad B7: unconnected-(J1-PadB7) -> sel1
- J1 pad B8: unconnected-(J1-PadB8) -> sel0
- J1 pad B9: VBUS -> sel3
- J3 pad 1: osc_out -> +3.3V
- J3 pad 2: xclk -> USER_RST
- J4 pad 1: Caravel_CSB -> Net-(J4-Pin_1)
- J4 pad 2: Caravel_SCK -> GND
- J4 pad 3: Caravel_D0 -> Net-(J4-Pin_3)
- J5 pad 1: GND -> osc_out
- J5 pad 2: mprj_io[8] -> xclk
- J5 pad 3: mprj_io[9] -> ext_clk
- J6 pad 1: mprj_io[19] -> Caravel_CSB
- J6 pad 2: mprj_io[20] -> Caravel_SCK
- J6 pad 3: mprj_io[21] -> Caravel_D0
- J6 pad 4: mprj_io[22] -> Caravel_D1
- J6 pad 5: mprj_io[23] -> +3.3V
- J6 pad 6: mprj_io[24] -> GND
- J7 pad 1: ~{MRST} -> GND
- J7 pad 2: GND -> scansel0
- R1 pad 1: Net-(J1-PadB5) -> Net-(J2-CC2)
- R10 pad 1: vdda -> +3.3V
- R12 pad 1: vdda -> +3.3V
- R13 pad 1: vccd -> +1V8
- R14 pad 1: vdda -> +3.3V
- R2 pad 1: Net-(J1-PadA5) -> Net-(J2-CC1)
- R3 pad 1: vdda -> +3.3V
- R4 pad 1: vdda -> +3.3V
- R5 pad 1: vccd -> Net-(J2-SHIELD)
- R5 pad 2: Net-(R5-Pad2) -> GND
- R6 pad 2: GND -> +3.3V
- R7 pad 1: vdda -> +3.3V
- R8 pad 1: vdda -> +3.3V
- R9 pad 1: vdda -> +3.3V
- SW1 pad 1: ~{MRST} -> USER_RST
- SW1 pad 2: GND -> +3.3V
- TP2 pad 1: vdda -> +3.3V
- TP3 pad 1: vccd -> +1V8
- U1 pad 1: ~{MRST} -> Net-(U1-GPIO0)
- U1 pad 27: rpi_clk -> ext_clk
- U1 pad 41: unconnected-(U5-Pad41) -> Net-(J4-Pin_3)
- U1 pad 43: unconnected-(U5-Pad43) -> Net-(J4-Pin_1)
- U3 pad 2: vdda -> +3.3V
- U4 pad 8: vdda -> +3.3V
- X1 pad 4: vdda -> +3.3V
Routing:
- net GND: track 566.7 -> 0.00 mm, vias 175 -> 0
- net vdda: track 242.7 -> 0.00 mm, vias 7 -> 0
- net Caravel_CSB: track 106.9 -> 0.00 mm, vias 2 -> 0
- net Caravel_SCK: track 100.4 -> 0.00 mm, vias 2 -> 0
- net Caravel_D0: track 99.1 -> 0.00 mm, vias 2 -> 0
- net vccd: track 98.5 -> 0.00 mm, vias 6 -> 0
- net Caravel_D1: track 93.1 -> 0.00 mm, vias 2 -> 0
- net xclk: track 67.9 -> 0.00 mm, vias 2 -> 0
- net rpi_clk: track 61.3 -> 0.00 mm, vias 3 -> 0
- net +5V: track 54.8 -> 0.00 mm, vias 3 -> 0
- net mprj_io[18]: track 50.6 -> 0.00 mm, vias 1 -> 0
- net mprj_io[16]: track 49.9 -> 0.00 mm
- net mprj_io[14]: track 49.9 -> 0.00 mm
- net mprj_io[12]: track 48.8 -> 0.00 mm
- net mprj_io[8]: track 47.8 -> 0.00 mm
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- removed copper zone on B.Cu, net GND
- removed copper zone on F.Cu, net GND
Other:
- board outline removed

Commit message: prelim floorplan done
Parts:
- moved kibuzzard-63FCFA05 213.2 mm to (148.3, 95.6), turned to 180 degrees
- moved R35 211.6 mm to (68.0, 90.0), turned to -90 degrees
- moved kibuzzard-63FCF9FA 211.2 mm to (148.3, 93.1), turned to 180 degrees
- moved kibuzzard-63FCF9EA 209.3 mm to (148.3, 90.6), turned to 180 degrees
- moved kibuzzard-63FCF9E0 207.3 mm to (148.3, 88.0), turned to 180 degrees
- moved kibuzzard-63FCF9CF 205.4 mm to (148.3, 85.4), turned to 180 degrees
- moved kibuzzard-63FCFA48 203.6 mm to (148.3, 82.9), turned to 180 degrees
- moved kibuzzard-64031BAD 203.1 mm to (146.8, 79.6), turned to 180 degrees
- moved D1 197.7 mm to (142.5, 57.6), turned to 90 degrees
- moved kibuzzard-6403978F 197.5 mm to (82.1, 60.2), turned to -90 degrees
- moved R22 195.6 mm to (141.0, 57.6), turned to 90 degrees
- moved D2 193.4 mm to (137.5, 57.5), turned to 90 degrees
- moved kibuzzard-63FE0946 193.4 mm to (61.5, 114.3)
- moved kibuzzard-63FE0972 193.4 mm to (61.5, 63.5)
- moved kibuzzard-63FE0972 193.4 mm to (61.5, 116.8)
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- renumbered C2 to C1, C6 to C10, C34 to C11, C8 to C12, C35 to C13, C25 to C14, C31 to C15, C20 to C16, C21 to C17, C24 to C18, C26 to C19, C29 to C2, C23 to C20, C19 to C21, C32 to C23, C27 to C24, C18 to C25, C28 to C26, C30 to C3, C9 to C6, C3 to C8, C33 to C9, J6 to J1, J7 to J10, J8 to J11, J11 to J2, J10 to J3, J3 to J4, J2 to J6, J1 to J7, J4 to J8, R30 to R1, R49 to R10, R5 to R11, R3 to R12, R4 to R13, R1 to R14, R2 to R15, R7 to R16, R8 to R17, R9 to R18, R10 to R19, R29 to R2, R34 to R20, R32 to R21, R11 to R22, R12 to R23, R31 to R24, R13 to R25, R15 to R26, R16 to R27, R17 to R28, R18 to R29, R28 to R3, R19 to R30, R20 to R31, R21 to R32, R22 to R33, R14 to R34, R39 to R35, R27 to R4, R26 to R5, R25 to R6, R6 to R7, R24 to R8, R23 to R9, SW5 to SW1, SW3 to SW2, SW1 to SW3, SW2 to SW4, TP11 to TP1, TP1 to TP10, TP5 to TP11, TP2 to TP12, TP3 to TP13, TP12 to TP2, TP13 to TP3, TP7 to TP4, TP8 to TP5, TP9 to TP6, TP10 to TP7, TP6 to TP8, TP4 to TP9, U4 to U1, U3 to U2, U6 to U3, U1 to U4, U7 to U5
Other:
- board outline added: 107.5 x 81 mm
- board text added: "0"
- board text added: "1"
- board text added: "2"
- board text added: "3"
- board text added: "4"
- board text added: "5"
- board text added: "6"
- board text added: "7"
- board text added: "8"
- board text added: "I/O PMODs"
- board text added: "Input"
- board text added: "Output"
- board text added: "Select Project"
- board text added: "TT motherboard: PRELIMINARY"
- board text removed: "MB1 rev A"

Commit message: pre-routing
Parts:
- removed the TP1 at (138.5, 78.8)
- removed the TP2 at (133.1, 94.5)
- removed the TP6 at (136.7, 98.3)
- removed the TP7 at (141.1, 82.7)
- removed TP9: Keystone 5019, TestPoint:TestPoint_Keystone_5019_Minature
- J10, J11: value Conn_01x22 -> Conn_01x24; footprint Connector_PinHeader_2.54mm:PinHeader_1x22_P2.54mm_Vertical -> Connector_PinHeader_2.54mm:PinHeader_1x24_P2.54mm_Vertical
- moved J8 80.3 mm to (27.4, 80.2), turned to 0 degrees
- moved X1 68.4 mm to (147.8, 64.6), turned to 180 degrees
- moved C5 67.9 mm to (147.2, 67.8), turned to 90 degrees
- moved TP1 66.8 mm to (147.7, 61.0), turned to 0 degrees
- moved kibuzzard-6403978F 59.7 mm to (141.5, 66.0)
- moved J5 59.5 mm to (144.2, 63.7), turned to 0 degrees
- moved C15 47.0 mm to (79.5, 64.3)
- moved C14 47.0 mm to (81.0, 64.3)
- moved C12 28.3 mm to (148.4, 131.2), turned to -90 degrees
- moved C10 26.1 mm to (146.6, 131.1), turned to -90 degrees
- moved C8 24.5 mm to (134.5, 131.0), turned to 90 degrees
- moved JP2 22.9 mm to (147.0, 99.0), turned to 180 degrees
- moved JP3 22.9 mm to (147.0, 101.5), turned to 180 degrees
- moved JP4 22.9 mm to (147.0, 104.0), turned to 180 degrees
- moved JP5 22.9 mm to (147.0, 106.5), turned to 180 degrees
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- renumbered TP3 to TP1, TP8 to TP2, TP5 to TP3, TP11 to TP5, TP10 to TP6, TP12 to TP7, TP13 to TP8
Connections:
- J10 pad 10: sel4 -> sel5
- J10 pad 11: sel5 -> sel6
- J10 pad 12: sel6 -> sel7
- J10 pad 13: mprj_io7 -> sel8
- J10 pad 14: mprj_io6_ser_tx -> set_clk_div
- J10 pad 15: mprj_io5_ser_rx -> slow_clk
- J10 pad 16: mprj_io4_SCK -> in0
- J10 pad 17: mprj_io3_CSB -> in1
- J10 pad 18: mprj_io2_SDI -> in2
- J10 pad 19: mprj_io1_SDO -> in3
- J10 pad 2: scansel0 -> +5V
- J10 pad 20: mprj_io0 -> in4
- J10 pad 21: +3.3V -> in5
- J10 pad 22: GND -> in6
- J10 pad 3: scansel1 -> scansel0
- J10 pad 4: slow_clk -> scansel1
- J10 pad 5: set_clk_div -> sel0
- J10 pad 6: sel0 -> sel1
- J10 pad 7: sel1 -> sel2
- J10 pad 8: sel2 -> sel3
- J10 pad 9: sel3 -> sel4
- J11 pad 1: sel7 -> GND
- J11 pad 10: in7 -> mprj_io6_ser_tx
- J11 pad 11: out0 -> mprj_io7
- J11 pad 12: out1 -> GND
- J11 pad 13: out2 -> out0
- J11 pad 14: out3 -> out1
- J11 pad 15: out4 -> out2
- J11 pad 16: out5 -> out3
- J11 pad 17: out6 -> out4
- J11 pad 18: out7 -> out5
- J11 pad 19: ready -> out6
- J11 pad 2: sel8 -> ext_clk
- J11 pad 20: +3.3V -> out7
- J11 pad 21: +5V -> GND
- J11 pad 22: GND -> +1V8
- J11 pad 3: in0 -> ready
- J11 pad 4: in1 -> mprj_io0
- J11 pad 5: in2 -> mprj_io1_SDO
- J11 pad 6: in3 -> mprj_io2_SDI
- J11 pad 7: in4 -> mprj_io3_CSB
- J11 pad 8: in5 -> mprj_io4_SCK
- J11 pad 9: in6 -> mprj_io5_ser_rx
- RN2 pad 10: in6 -> in1
- RN2 pad 11: in5 -> in2
- RN2 pad 12: in4 -> in3
- RN2 pad 13: in3 -> in4
- RN2 pad 14: in2 -> in5
- RN2 pad 15: in1 -> in6
- RN2 pad 16: in0 -> in7
- RN2 pad 9: in7 -> in0
Routing:
- net +3.3V: track 0.00 -> 21.8 mm, vias 0 -> 2
- added copper zone on B.Cu, net GND
- added copper zone on F.Cu, net GND
Other:
- board size 107.5 x 81 mm -> 104.5 x 81 mm
- board text added: "TODO: PIN LABELS"

Commit message: v2.0 alpha, routing complete
Parts:
- removed J8: Conn_01x03, Connector_PinHeader_2.54mm:PinHeader_1x03_P2.54mm_Vertical
- removed TP1: TestPoint, TestPoint:TestPoint_Pad_D1.5mm
- removed kibuzzard-63FE0746: G***, kibuzzard-63FE0746
- removed kibuzzard-63FE0751: G***, kibuzzard-63FE0751
- removed kibuzzard-63FE075A: G***, kibuzzard-63FE075A
- removed kibuzzard-63FE076E: G***, kibuzzard-63FE076E
- removed kibuzzard-63FE0776: G***, kibuzzard-63FE0776
- removed kibuzzard-63FE0780: G***, kibuzzard-63FE0780
- removed kibuzzard-63FE078B: G***, kibuzzard-63FE078B
- removed kibuzzard-63FE0797: G***, kibuzzard-63FE0797
- removed kibuzzard-63FE080F: G***, kibuzzard-63FE080F
- removed kibuzzard-63FE0813: G***, kibuzzard-63FE0813
- removed kibuzzard-63FE0819: G***, kibuzzard-63FE0819
- removed kibuzzard-63FE081F: G***, kibuzzard-63FE081F
- removed kibuzzard-63FE0824: G***, kibuzzard-63FE0824
- removed kibuzzard-63FE0829: G***, kibuzzard-63FE0829
- removed kibuzzard-63FE0830: G***, kibuzzard-63FE0830
- removed kibuzzard-63FE0835: G***, kibuzzard-63FE0835
- removed kibuzzard-63FE083A: G***, kibuzzard-63FE083A
- removed kibuzzard-63FE083F: G***, kibuzzard-63FE083F
- removed kibuzzard-63FE0946 (x2): G***, kibuzzard-63FE0946
- removed kibuzzard-63FE0967: G***, kibuzzard-63FE0967
- removed kibuzzard-63FE0972 (x3): G***, kibuzzard-63FE0972
- removed kibuzzard-63FE09CE: G***, kibuzzard-63FE09CE
- removed kibuzzard-63FE09E3: G***, kibuzzard-63FE09E3
- removed kibuzzard-63FE09F3: G***, kibuzzard-63FE09F3
- removed kibuzzard-63FE09FD: G***, kibuzzard-63FE09FD
- removed kibuzzard-63FE0A06: G***, kibuzzard-63FE0A06
- removed kibuzzard-63FE0A17: G***, kibuzzard-63FE0A17
- removed kibuzzard-63FE0A28: G***, kibuzzard-63FE0A28
- removed kibuzzard-63FE0A36: G***, kibuzzard-63FE0A36
- removed kibuzzard-63FE0A4C: G***, kibuzzard-63FE0A4C
- removed kibuzzard-63FE0A5C: G***, kibuzzard-63FE0A5C
- removed kibuzzard-63FE0A7D: G***, kibuzzard-63FE0A7D
- removed kibuzzard-63FE0A8A: G***, kibuzzard-63FE0A8A
- removed kibuzzard-63FE0AA2: G***, kibuzzard-63FE0AA2
- removed kibuzzard-63FE0AAA: G***, kibuzzard-63FE0AAA
- removed kibuzzard-63FE0AB4: G***, kibuzzard-63FE0AB4
- removed kibuzzard-63FE0AC0: G***, kibuzzard-63FE0AC0
- removed kibuzzard-63FE0AC9: G***, kibuzzard-63FE0AC9
- removed kibuzzard-63FE0AD7: G***, kibuzzard-63FE0AD7
- removed kibuzzard-63FE0AE3: G***, kibuzzard-63FE0AE3
- removed kibuzzard-63FE4154: G***, kibuzzard-63FE4154
- removed kibuzzard-6403978F: G***, kibuzzard-6403978F
- added G***: LOGO, flyingcarsfootprints:PsychoLogo, B.Cu at (108.0, 118.2)
- added REF**: TT_logo, Logos:TT_logo, F.Cu at (107.2, 63.2)
- added REF**: Logo, Logos:ef_logo_graphical, F.Cu at (107.5, 93.5)
- added REF**: Logo, Logos:ef_logo, F.Cu at (107.5, 98.0)
- added REF**: Z2A_logo, Logos:Z2A_logo, F.Cu at (107.2, 110.5)
- added STITCH: StitchingVia-0.4mmDrill, flyingcarsfootprints:StitchingVia-0.4mmDrill, F.Cu at (96.6, 118.9)
- added STITCH: StitchingVia-0.4mmDrill, flyingcarsfootprints:StitchingVia-0.4mmDrill, F.Cu at (135.0, 97.3)
- added STITCH: StitchingVia-0.4mmDrill, flyingcarsfootprints:StitchingVia-0.4mmDrill, F.Cu at (146.0, 90.5)
- added STITCH: StitchingVia-0.4mmDrill, flyingcarsfootprints:StitchingVia-0.4mmDrill, F.Cu at (60.4, 70.3)
- added STITCH: StitchingVia-0.4mmDrill, flyingcarsfootprints:StitchingVia-0.4mmDrill, F.Cu at (60.4, 77.9)
- added STITCH: StitchingVia-0.4mmDrill, flyingcarsfootprints:StitchingVia-0.4mmDrill, F.Cu at (92.2, 55.3)
- added STITCH: StitchingVia-0.4mmDrill, flyingcarsfootprints:StitchingVia-0.4mmDrill, F.Cu at (152.6, 86.3)
- added STITCH: StitchingVia-0.4mmDrill, flyingcarsfootprints:StitchingVia-0.4mmDrill, F.Cu at (114.8, 120.7)
- added STITCH: StitchingVia-0.4mmDrill, flyingcarsfootprints:StitchingVia-0.4mmDrill, F.Cu at (64.8, 105.9)
- added STITCH: StitchingVia-0.4mmDrill, flyingcarsfootprints:StitchingVia-0.4mmDrill, F.Cu at (88.8, 92.1)
- added STITCH: StitchingVia-0.4mmDrill, flyingcarsfootprints:StitchingVia-0.4mmDrill, F.Cu at (86.2, 117.7)
- added STITCH: StitchingVia-0.4mmDrill, flyingcarsfootprints:StitchingVia-0.4mmDrill, F.Cu at (146.6, 79.5)
- added STITCH: StitchingVia-0.4mmDrill, flyingcarsfootprints:StitchingVia-0.4mmDrill, F.Cu at (78.4, 65.7)
- added STITCH: StitchingVia-0.4mmDrill, flyingcarsfootprints:StitchingVia-0.4mmDrill, F.Cu at (70.2, 89.1)
- added STITCH: StitchingVia-0.4mmDrill, flyingcarsfootprints:StitchingVia-0.4mmDrill, F.Cu at (115.0, 116.9)
- added STITCH: StitchingVia-0.4mmDrill, flyingcarsfootprints:StitchingVia-0.4mmDrill, F.Cu at (89.0, 69.3)
- added STITCH: StitchingVia-0.4mmDrill, flyingcarsfootprints:StitchingVia-0.4mmDrill, F.Cu at (104.8, 81.9)
- added STITCH: StitchingVia-0.4mmDrill, flyingcarsfootprints:StitchingVia-0.4mmDrill, F.Cu at (91.6, 67.9)
- added STITCH: StitchingVia-0.4mmDrill, flyingcarsfootprints:StitchingVia-0.4mmDrill, F.Cu at (114.4, 99.9)
- added STITCH: StitchingVia-0.4mmDrill, flyingcarsfootprints:StitchingVia-0.4mmDrill, F.Cu at (71.4, 85.7)
- added STITCH: StitchingVia-0.4mmDrill, flyingcarsfootprints:StitchingVia-0.4mmDrill, F.Cu at (111.8, 64.9)
- added STITCH: StitchingVia-0.4mmDrill, flyingcarsfootprints:StitchingVia-0.4mmDrill, F.Cu at (129.6, 97.3)
- added STITCH: StitchingVia-0.4mmDrill, flyingcarsfootprints:StitchingVia-0.4mmDrill, F.Cu at (147.8, 62.3)
- added STITCH: StitchingVia-0.4mmDrill, flyingcarsfootprints:StitchingVia-0.4mmDrill, F.Cu at (66.2, 101.3)
- added STITCH: StitchingVia-0.4mmDrill, flyingcarsfootprints:StitchingVia-0.4mmDrill, F.Cu at (83.2, 108.5)
- added STITCH: StitchingVia-0.4mmDrill, flyingcarsfootprints:StitchingVia-0.4mmDrill, F.Cu at (126.0, 59.5)
- added STITCH: StitchingVia-0.4mmDrill, flyingcarsfootprints:StitchingVia-0.4mmDrill, F.Cu at (83.0, 57.0)
- added STITCH: StitchingVia-0.4mmDrill, flyingcarsfootprints:StitchingVia-0.4mmDrill, F.Cu at (75.0, 121.9)
- added STITCH: StitchingVia-0.4mmDrill, flyingcarsfootprints:StitchingVia-0.4mmDrill, F.Cu at (104.8, 88.3)
- added STITCH: StitchingVia-0.4mmDrill, flyingcarsfootprints:StitchingVia-0.4mmDrill, F.Cu at (134.4, 67.1)
- added STITCH: StitchingVia-0.4mmDrill, flyingcarsfootprints:StitchingVia-0.4mmDrill, F.Cu at (66.6, 96.3)
- added STITCH: StitchingVia-0.4mmDrill, flyingcarsfootprints:StitchingVia-0.4mmDrill, F.Cu at (68.2, 67.9)
- added STITCH: StitchingVia-0.4mmDrill, flyingcarsfootprints:StitchingVia-0.4mmDrill, F.Cu at (72.8, 75.7)
- added STITCH: StitchingVia-0.4mmDrill, flyingcarsfootprints:StitchingVia-0.4mmDrill, F.Cu at (68.4, 72.9)
- added STITCH: StitchingVia-0.4mmDrill, flyingcarsfootprints:StitchingVia-0.4mmDrill, F.Cu at (110.6, 93.5)
- added STITCH: StitchingVia-0.4mmDrill, flyingcarsfootprints:StitchingVia-0.4mmDrill, F.Cu at (94.0, 104.7)
- added STITCH: StitchingVia-0.4mmDrill, flyingcarsfootprints:StitchingVia-0.4mmDrill, F.Cu at (123.8, 57.3)
- added STITCH: StitchingVia-0.4mmDrill, flyingcarsfootprints:StitchingVia-0.4mmDrill, F.Cu at (153.6, 95.5)
- added STITCH: StitchingVia-0.4mmDrill, flyingcarsfootprints:StitchingVia-0.4mmDrill, F.Cu at (57.2, 62.7)
- added STITCH: StitchingVia-0.4mmDrill, flyingcarsfootprints:StitchingVia-0.4mmDrill, F.Cu at (65.4, 121.9)
- added STITCH: StitchingVia-0.4mmDrill, flyingcarsfootprints:StitchingVia-0.4mmDrill, F.Cu at (122.8, 64.9)
- added STITCH: StitchingVia-0.4mmDrill, flyingcarsfootprints:StitchingVia-0.4mmDrill, F.Cu at (140.8, 68.5)
- added STITCH: StitchingVia-0.4mmDrill, flyingcarsfootprints:StitchingVia-0.4mmDrill, F.Cu at (91.6, 119.1)
- added STITCH: StitchingVia-0.4mmDrill, flyingcarsfootprints:StitchingVia-0.4mmDrill, F.Cu at (102.4, 64.9)
- added STITCH: StitchingVia-0.4mmDrill, flyingcarsfootprints:StitchingVia-0.4mmDrill, F.Cu at (153.2, 75.1)
- added STITCH: StitchingVia-0.4mmDrill, flyingcarsfootprints:StitchingVia-0.4mmDrill, F.Cu at (115.0, 111.7)
- added STITCH: StitchingVia-0.4mmDrill, flyingcarsfootprints:StitchingVia-0.4mmDrill, F.Cu at (149.0, 68.5)
- added STITCH: StitchingVia-0.4mmDrill, flyingcarsfootprints:StitchingVia-0.4mmDrill, F.Cu at (68.4, 80.5)
- added STITCH: StitchingVia-0.4mmDrill, flyingcarsfootprints:StitchingVia-0.4mmDrill, F.Cu at (102.4, 71.5)
- added STITCH: StitchingVia-0.4mmDrill, flyingcarsfootprints:StitchingVia-0.4mmDrill, F.Cu at (78.4, 80.7)
- added STITCH: StitchingVia-0.4mmDrill, flyingcarsfootprints:StitchingVia-0.4mmDrill, F.Cu at (65.4, 111.1)
- added STITCH: StitchingVia-0.4mmDrill, flyingcarsfootprints:StitchingVia-0.4mmDrill, F.Cu at (101.2, 55.1)
- added STITCH: StitchingVia-0.4mmDrill, flyingcarsfootprints:StitchingVia-0.4mmDrill, F.Cu at (104.8, 94.9)
- added STITCH: StitchingVia-0.4mmDrill, flyingcarsfootprints:StitchingVia-0.4mmDrill, F.Cu at (69.2, 54.3)
- added STITCH1: StitchingVia-0.4mmDrill, flyingcarsfootprints:StitchingVia-0.4mmDrill, F.Cu at (104.2, 55.1)
- added STITCH10: StitchingVia-0.4mmDrill, flyingcarsfootprints:StitchingVia-0.4mmDrill, F.Cu at (145.0, 133.7)
- added STITCH11: StitchingVia-0.4mmDrill, flyingcarsfootprints:StitchingVia-0.4mmDrill, F.Cu at (140.0, 133.7)
- added STITCH12: StitchingVia-0.4mmDrill, flyingcarsfootprints:StitchingVia-0.4mmDrill, F.Cu at (135.0, 133.7)
- added STITCH13: StitchingVia-0.4mmDrill, flyingcarsfootprints:StitchingVia-0.4mmDrill, F.Cu at (130.0, 133.7)
- added STITCH14: StitchingVia-0.4mmDrill, flyingcarsfootprints:StitchingVia-0.4mmDrill, F.Cu at (125.0, 133.7)
- added STITCH15: StitchingVia-0.4mmDrill, flyingcarsfootprints:StitchingVia-0.4mmDrill, F.Cu at (120.0, 133.7)
- added STITCH16: StitchingVia-0.4mmDrill, flyingcarsfootprints:StitchingVia-0.4mmDrill, F.Cu at (115.0, 133.7)
- added STITCH17: StitchingVia-0.4mmDrill, flyingcarsfootprints:StitchingVia-0.4mmDrill, F.Cu at (108.6, 125.1)
- added STITCH17: StitchingVia-0.4mmDrill, flyingcarsfootprints:StitchingVia-0.4mmDrill, F.Cu at (110.0, 133.7)
- added STITCH18: StitchingVia-0.4mmDrill, flyingcarsfootprints:StitchingVia-0.4mmDrill, F.Cu at (105.0, 133.7)
- added STITCH19: StitchingVia-0.4mmDrill, flyingcarsfootprints:StitchingVia-0.4mmDrill, F.Cu at (108.6, 120.1)
- added STITCH2: StitchingVia-0.4mmDrill, flyingcarsfootprints:StitchingVia-0.4mmDrill, F.Cu at (107.2, 55.1)
- added STITCH20: StitchingVia-0.4mmDrill, flyingcarsfootprints:StitchingVia-0.4mmDrill, F.Cu at (108.6, 115.1)
- added STITCH21: StitchingVia-0.4mmDrill, flyingcarsfootprints:StitchingVia-0.4mmDrill, F.Cu at (90.0, 133.7)
- added STITCH22: StitchingVia-0.4mmDrill, flyingcarsfootprints:StitchingVia-0.4mmDrill, F.Cu at (85.0, 133.7)
- added STITCH23: StitchingVia-0.4mmDrill, flyingcarsfootprints:StitchingVia-0.4mmDrill, F.Cu at (80.0, 133.7)
- added STITCH24: StitchingVia-0.4mmDrill, flyingcarsfootprints:StitchingVia-0.4mmDrill, F.Cu at (108.6, 110.1)
- added STITCH25: StitchingVia-0.4mmDrill, flyingcarsfootprints:StitchingVia-0.4mmDrill, F.Cu at (72.0, 133.7)
- added STITCH25: StitchingVia-0.4mmDrill, flyingcarsfootprints:StitchingVia-0.4mmDrill, F.Cu at (67.6, 133.7)
- added STITCH27: StitchingVia-0.4mmDrill, flyingcarsfootprints:StitchingVia-0.4mmDrill, F.Cu at (108.6, 100.1)
- added STITCH28: StitchingVia-0.4mmDrill, flyingcarsfootprints:StitchingVia-0.4mmDrill, F.Cu at (108.6, 95.1)
- added STITCH29: StitchingVia-0.4mmDrill, flyingcarsfootprints:StitchingVia-0.4mmDrill, F.Cu at (108.6, 90.1)
- added STITCH3: StitchingVia-0.4mmDrill, flyingcarsfootprints:StitchingVia-0.4mmDrill, F.Cu at (110.2, 55.1)
- added STITCH30: StitchingVia-0.4mmDrill, flyingcarsfootprints:StitchingVia-0.4mmDrill, F.Cu at (108.6, 85.5)
- added STITCH32: StitchingVia-0.4mmDrill, flyingcarsfootprints:StitchingVia-0.4mmDrill, F.Cu at (108.6, 75.1)
- added STITCH33: StitchingVia-0.4mmDrill, flyingcarsfootprints:StitchingVia-0.4mmDrill, F.Cu at (108.6, 70.1)
- added STITCH34: StitchingVia-0.4mmDrill, flyingcarsfootprints:StitchingVia-0.4mmDrill, F.Cu at (108.6, 65.1)
- added STITCH35: StitchingVia-0.4mmDrill, flyingcarsfootprints:StitchingVia-0.4mmDrill, F.Cu at (87.0, 58.9)
- added STITCH4: StitchingVia-0.4mmDrill, flyingcarsfootprints:StitchingVia-0.4mmDrill, F.Cu at (113.2, 55.1)
- added STITCH4: StitchingVia-0.4mmDrill, flyingcarsfootprints:StitchingVia-0.4mmDrill, F.Cu at (125.0, 54.3)
- added STITCH5: StitchingVia-0.4mmDrill, flyingcarsfootprints:StitchingVia-0.4mmDrill, F.Cu at (130.0, 54.3)
- added STITCH6: StitchingVia-0.4mmDrill, flyingcarsfootprints:StitchingVia-0.4mmDrill, F.Cu at (135.0, 54.3)
- added STITCH7: StitchingVia-0.4mmDrill, flyingcarsfootprints:StitchingVia-0.4mmDrill, F.Cu at (140.0, 54.3)
- added STITCH8: StitchingVia-0.4mmDrill, flyingcarsfootprints:StitchingVia-0.4mmDrill, F.Cu at (145.0, 54.3)
- added STITCH9: StitchingVia-0.4mmDrill, flyingcarsfootprints:StitchingVia-0.4mmDrill, F.Cu at (150.0, 133.7)
- added STITCH9: StitchingVia-0.4mmDrill, flyingcarsfootprints:StitchingVia-0.4mmDrill, F.Cu at (150.0, 54.3)
- moved G*** 30.5 mm to (107.2, 78.0)
- moved G*** 30.5 mm to (107.2, 82.8)
- moved kibuzzard-64031BAD 18.3 mm to (146.4, 71.3), turned to 0 degrees
- moved RN2 17.6 mm to (75.2, 63.0), turned to -90 degrees
- moved TP6 8.75 mm to (77.2, 125.2), turned to 90 degrees
- moved TP4 8.59 mm to (140.2, 78.5)
- moved R34 5.80 mm to (133.2, 63.5), turned to -90 degrees
- moved C4 3.58 mm to (62.8, 126.2), turned to 180 degrees
- moved TP2 3.10 mm to (78.0, 58.0)
- moved R35 2.80 mm to (66.5, 89.8), turned to 180 degrees
- moved J10 2.54 mm to (58.6, 124.7)
- moved J11 2.54 mm to (157.8, 66.2)
- moved C14 2.49 mm to (80.0, 62.0)
- moved C15 2.49 mm to (78.5, 62.0)
- moved RN1 1.86 mm to (87.5, 105.0)
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Connections:
- J10 pad 10: sel5 -> sel3
- J10 pad 11: sel6 -> sel4
- J10 pad 12: sel7 -> sel5
- J10 pad 13: sel8 -> sel6
- J10 pad 14: set_clk_div -> sel7
- J10 pad 15: slow_clk -> sel8
- J10 pad 5: sel0 -> set_clk_div
- J10 pad 6: sel1 -> slow_clk
- J10 pad 7: sel2 -> sel0
- J10 pad 8: sel3 -> sel1
- J10 pad 9: sel4 -> sel2
- U4 pad 10: unconnected-(U4-GPIO7-Pad10) -> out2
- U4 pad 11: unconnected-(U4-GPIO8-Pad11) -> out1
- U4 pad 12: unconnected-(U4-GPIO9-Pad12) -> out0
- U4 pad 19: unconnected-(U4-GPIO14-Pad19) -> in0
- U4 pad 20: unconnected-(U4-GPIO15-Pad20) -> in1
- U4 pad 21: unconnected-(U4-GPIO16-Pad21) -> in2
- U4 pad 22: unconnected-(U4-GPIO17-Pad22) -> in3
- U4 pad 24: unconnected-(U4-GPIO18-Pad24) -> in4
- U4 pad 25: unconnected-(U4-GPIO19-Pad25) -> in5
- U4 pad 26: unconnected-(U4-GPIO20-Pad26) -> in6
- U4 pad 27: ext_clk -> in7
- U4 pad 29: unconnected-(U4-GPIO22-Pad29) -> out4
- U4 pad 31: unconnected-(U4-GPIO26_ADC0-Pad31) -> out5
- U4 pad 32: unconnected-(U4-GPIO27_ADC1-Pad32) -> out6
- U4 pad 34: unconnected-(U4-GPIO28_ADC2-Pad34) -> out7
- U4 pad 7: unconnected-(U4-GPIO5-Pad7) -> ext_clk
- U4 pad 9: unconnected-(U4-GPIO6-Pad9) -> out3
Routing:
- net +3.3V: track 21.8 -> 509.4 mm, vias 2 -> 46
- net +5V: track 0.00 -> 192.0 mm, vias 0 -> 13
- net out7: track 0.00 -> 171.3 mm, vias 0 -> 6
- net out5: track 0.00 -> 159.9 mm, vias 0 -> 9
- net +1V8: track 0.00 -> 159.2 mm, vias 0 -> 8
- net out6: track 0.00 -> 158.9 mm, vias 0 -> 6
- net out3: track 0.00 -> 153.5 mm, vias 0 -> 7
- net out2: track 0.00 -> 143.9 mm, vias 0 -> 8
- net out4: track 0.00 -> 143.2 mm, vias 0 -> 7
- net out1: track 0.00 -> 140.6 mm, vias 0 -> 4
- net in0: track 0.00 -> 136.5 mm, vias 0 -> 10
- net in1: track 0.00 -> 134.2 mm, vias 0 -> 7
- net out0: track 0.00 -> 129.1 mm, vias 0 -> 4
- net in7: track 0.00 -> 127.6 mm, vias 0 -> 8
- net in4: track 0.00 -> 124.3 mm, vias 0 -> 8
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Other:
- board text added: "(C) 2023 Pat Deegan, https://psychogenic.com"
- board text added: "+5V"
- board text added: "1V8"
- board text added: "3V3"
- board text added: "3v3"
- board text added: "CLK"
- board text added: "CLK SEL"
- board text added: "CLKDv"
- board text added: "EXT"
- board text added: "ExCLK"
- board text added: "Ext"
- board text added: "GND"
- board text added: "Int"
- board text added: "Logic"
- board text added: "MIO0"
- board text added: "MIO1"
- board text added: "MIO2"
- board text added: "MIO3"
- board text added: "MIO4"
- board text added: "MIO5"
- board text added: "MIO6"
- board text added: "MIO7"
- board text added: "OSC"
- board text added: "RDY"
- board text added: "Raspberry Pi Pico"
- board text added: "SCAN SEL"
- board text added: "SCLK"
- board text added: "Scn0"
- board text added: "Scn1"
- board text added: "TinyTapeout Motherboard"
- board text added: "in0"
- board text added: "in1"
- board text added: "in2"
- board text added: "in3"
- board text added: "in4"
- board text added: "in5"
- board text added: "in6"
- board text added: "in7"
- board text added: "ot0"
- board text added: "ot1"
- board text added: "ot2"
- board text added: "ot3"
- board text added: "ot4"
- board text added: "ot5"
- board text added: "ot6"
- board text added: "ot7"
- board text added: "out0"
- board text added: "out1"
- board text added: "out2"
- board text added: "out3"
- board text added: "out4"
- board text added: "out5"
- board text added: "out6"
- board text added: "sel0"
- board text added: "sel1"
- board text added: "sel2"
- board text added: "sel3"
- board text added: "sel4"
- board text added: "sel5"
- board text added: "sel6"
- board text added: "sel7"
- board text added: "sel8"
- board text added: "v2.0"
- board text removed: "TODO: PIN LABELS"
- board text removed: "TT motherboard: PRELIMINARY"

Commit message: v2.1 release
Parts:
- removed STITCH19: StitchingVia-0.4mmDrill, flyingcarsfootprints:StitchingVia-0.4mmDrill
- removed kibuzzard-63FCF59C: G***, kibuzzard-63FCF59C
- removed kibuzzard-63FCF5C0: G***, kibuzzard-63FCF5C0
- removed kibuzzard-63FCF5C8: G***, kibuzzard-63FCF5C8
- removed kibuzzard-64048AFF: G***, kibuzzard-64048AFF
- removed kibuzzard-64048B08: G***, kibuzzard-64048B08
- removed kibuzzard-64048B12: G***, kibuzzard-64048B12
- removed kibuzzard-64048B21: G***, kibuzzard-64048B21
- added J8: Conn_01x02, Connector_PinHeader_2.54mm:PinHeader_1x02_P2.54mm_Vertical, F.Cu at (107.6, 118.3)
- added STITCH: StitchingVia-0.4mmDrill, flyingcarsfootprints:StitchingVia-0.4mmDrill, F.Cu at (72.8, 70.4)
- added STITCH: StitchingVia-0.4mmDrill, flyingcarsfootprints:StitchingVia-0.4mmDrill, F.Cu at (140.0, 127.0)
- added STITCH: StitchingVia-0.4mmDrill, flyingcarsfootprints:StitchingVia-0.4mmDrill, F.Cu at (139.1, 114.0)
- added STITCH: StitchingVia-0.4mmDrill, flyingcarsfootprints:StitchingVia-0.4mmDrill, F.Cu at (140.0, 120.5)
- added STITCH: StitchingVia-0.4mmDrill, flyingcarsfootprints:StitchingVia-0.4mmDrill, F.Cu at (117.7, 114.0)
- added STITCH: StitchingVia-0.4mmDrill, flyingcarsfootprints:StitchingVia-0.4mmDrill, F.Cu at (133.2, 114.0)
- added STITCH: StitchingVia-0.4mmDrill, flyingcarsfootprints:StitchingVia-0.4mmDrill, F.Cu at (124.2, 120.7)
- moved G*** 46.9 mm to (80.8, 80.0)
- moved REF** 0.59 mm to (107.2, 109.9)
Routing:
- net GND: track 110.7 -> 133.7 mm, vias 43 -> 50
- net Net-(J8-Pin_1): track 0.00 -> 15.8 mm
- net Net-(J8-Pin_2): track 0.00 -> 15.3 mm
- net set_clk_div: track 51.3 -> 52.6 mm
- net +3.3V: track 509.4 -> 510.3 mm
- net in7: track 127.6 -> 126.8 mm
- net slow_clk: track 50.5 -> 49.9 mm
- net Net-(U5-E): track 13.0 -> 13.5 mm
- net sel7: track 50.2 -> 49.7 mm
Other:
- board text added: "(C) 2023 Pat Deegan https://psychogenic.com"
- board text added: "2-layer, basic PCB 0.3mm drill min >6mil traces"
- board text added: "TODO: TP paste fp"
- board text added: "out7"
- board text added: "v2.1"
- board text removed: "(C) 2023 Pat Deegan, https://psychogenic.com"
- board text removed: "10MHz"
- board text removed: "Pico CLK"
- board text removed: "v2.0"

Commit message: v2.1 prototype run
Other:
- board text removed: "TODO: TP paste fp"
Changed lines of the file:
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@@
     (fp_line (start 1.9 0.5) (end 1.9 -0.5)
       (stroke (width 0.15) (type solid)) (layer "F.Fab"))
-    (pad "1" smd rect (at 0 0) (size 3.8 2) (layers "F.Cu" "F.Mask")
+    (pad "1" smd rect (at 0 0) (size 3.8 2) (layers "F.Cu" "F.Paste" "F.Mask")
       (net 10 "+3.3V") (pinfunction "1") (pintype "passive"))
     (model "${KICAD6_3DMODEL_DIR}/TestPoint.3dshapes/TestPoint_Keystone_5019_Minature.wrl"
@@
     (fp_line (start 1.9 0.5) (end 1.9 -0.5)
       (stroke (width 0.15) (type solid)) (layer "F.Fab"))
-    (pad "1" smd rect (at 0 0 270) (size 3.8 2) (layers "F.Cu" "F.Mask")
+    (pad "1" smd rect (at 0 0 270) (size 3.8 2) (layers "F.Cu" "F.Paste" "F.Mask")
       (net 12 "+1V8") (pinfunction "1") (pintype "passive"))
     (model "${KICAD6_3DMODEL_DIR}/TestPoint.3dshapes/TestPoint_Keystone_5019_Minature.wrl"
@@
     (fp_line (start 1.9 0.5) (end 1.9 -0.5)
       (stroke (width 0.15) (type solid)) (layer "F.Fab"))
-    (pad "1" smd rect (at 0 0 90) (size 3.8 2) (layers "F.Cu" "F.Mask")
+    (pad "1" smd rect (at 0 0 90) (size 3.8 2) (layers "F.Cu" "F.Paste" "F.Mask")
       (net 2 "+5V") (pinfunction "1") (pintype "passive"))
     (model "${KICAD6_3DMODEL_DIR}/TestPoint.3dshapes/TestPoint_Keystone_5019_Minature.wrl"
@@
     (effects (font (size 1.2 1.2) (thickness 0.2) bold) (justify right bottom))
   )
-  (gr_text "TODO: TP paste fp" (at 56.9 146.7) (layer "User.1")
-    (effects (font (size 2 2) (thickness 0.3)) (justify left bottom))
-  )
   (gr_text "2-layer, basic PCB\n0.3mm drill min\n>6mil traces" (at 141.5 148.5) (layer "User.1")
